File: KiCad/base/base/base.kicad_pcb (KiCad board)
At the start: 2 copper layers, 133.6 x 74.9 mm, 2 parts

Commit message: various fixes and changes
Parts:
- moved G*** 97.4 mm to (193.8, 87.8)
- moved G*** 97.4 mm to (196.8, 87.8)
Other:
- board size 133.6 x 74.9 mm -> 114.5 x 89.1 mm

Commit message: .
.
Parts:
- removed the G*** at (196.8, 87.8)
- removed the G*** at (193.8, 87.8)
- added G***: LOGO, Footprints:nd-x-lg-exposed-copper, B.Cu at (196.9, 87.8)
- added G***: LOGO, Footprints:nd-x-lg-exposed-copper, F.Cu at (193.9, 87.8)
- added REF**: MountingHole_2.2mm_M2_Pad_Via, MountingHole:MountingHole_2.2mm_M2_Pad_Via, F.Cu at (144.5, 120.8)
- added REF**: MountingHole_2.2mm_M2_Pad_Via, MountingHole:MountingHole_2.2mm_M2_Pad_Via, F.Cu at (225.4, 135.1)
- added REF**: MountingHole_2.2mm_M2_Pad_Via, MountingHole:MountingHole_2.2mm_M2_Pad_Via, F.Cu at (251.1, 135.1)
- added REF**: MountingHole_2.2mm_M2_Pad_Via, MountingHole:MountingHole_2.2mm_M2_Pad_Via, F.Cu at (246.2, 54.0)
- added REF**: MountingHole_2.2mm_M2_Pad_Via, MountingHole:MountingHole_2.2mm_M2_Pad_Via, F.Cu at (144.5, 54.0)
Routing:
- removed copper zone on B.Cu, net (none)
- removed copper zone on F.Cu, net (none)
Other:
- outline, holes or cut-outs redrawn
