File: KiCad/plate/Plate.kicad_pcb (KiCad board)
At the start: 2 copper layers, 133.6 x 74.9 mm, 0 parts

Commit message: various fixes and changes
Other:
- board size 133.6 x 74.9 mm -> 114.5 x 89.1 mm

Commit message: .
.
Parts:
- added REF**: MountingHole_2.2mm_M2_Pad_Via, MountingHole:MountingHole_2.2mm_M2_Pad_Via, F.Cu at (225.4, 135.1)
- added REF**: mx-alps-plated-cutout-reversible, Footprints:mx-alps-plated-cutout-reversible, F.Cu at (233.7, 103.0)
- added REF**: mx-alps-plated-cutout-reversible, Footprints:mx-alps-plated-cutout-reversible, F.Cu at (238.4, 122.1)
- added REF**: mx-alps-plated-cutout-reversible, Footprints:mx-alps-plated-cutout-reversible, F.Cu at (157.4, 84.0)
- added REF**: mx-alps-plated-cutout-reversible, Footprints:mx-alps-plated-cutout-reversible, F.Cu at (176.5, 84.0)
- added REF**: mx-alps-plated-cutout-reversible, Footprints:mx-alps-plated-cutout-reversible, F.Cu at (195.6, 84.0)
- added REF**: mx-alps-plated-cutout-reversible, Footprints:mx-alps-plated-cutout-reversible, F.Cu at (214.6, 84.0)
- added REF**: mx-alps-plated-cutout-reversible, Footprints:mx-alps-plated-cutout-reversible, F.Cu at (233.7, 84.0)
- added REF**: mx-alps-plated-cutout-reversible, Footprints:mx-alps-plated-cutout-reversible, F.Cu at (233.7, 65.0)
- added REF**: mx-alps-plated-cutout-reversible, Footprints:mx-alps-plated-cutout-reversible, F.Cu at (214.6, 65.0)
- added REF**: mx-alps-plated-cutout-reversible, Footprints:mx-alps-plated-cutout-reversible, F.Cu at (195.6, 65.0)
- added REF**: MountingHole_2.2mm_M2_Pad_Via, MountingHole:MountingHole_2.2mm_M2_Pad_Via, F.Cu at (251.1, 135.1)
- added REF**: mx-alps-plated-cutout-reversible, Footprints:mx-alps-plated-cutout-reversible, F.Cu at (176.5, 65.0)
- added REF**: mx-alps-plated-cutout-reversible, Footprints:mx-alps-plated-cutout-reversible, F.Cu at (157.4, 65.0)
- added REF**: MountingHole_2.2mm_M2_Pad_Via, MountingHole:MountingHole_2.2mm_M2_Pad_Via, F.Cu at (144.5, 120.8)
- added REF**: MountingHole_2.2mm_M2_Pad_Via, MountingHole:MountingHole_2.2mm_M2_Pad_Via, F.Cu at (246.2, 54.0)
- added REF**: MountingHole_2.2mm_M2_Pad_Via, MountingHole:MountingHole_2.2mm_M2_Pad_Via, F.Cu at (144.5, 54.0)
- added REF**: mx-alps-plated-cutout-reversible, Footprints:mx-alps-plated-cutout-reversible, F.Cu at (157.4, 103.1)
- added REF**: mx-alps-plated-cutout-reversible, Footprints:mx-alps-plated-cutout-reversible, F.Cu at (176.5, 103.0)
- added REF**: mx-alps-plated-cutout-reversible, Footprints:mx-alps-plated-cutout-reversible, F.Cu at (195.6, 103.1)
- added REF**: mx-alps-plated-cutout-reversible, Footprints:mx-alps-plated-cutout-reversible, F.Cu at (214.6, 103.1)
Routing:
- removed copper zone on B.Cu, net (none)
- removed copper zone on F.Cu, net (none)
Other:
- outline, holes or cut-outs redrawn
