File: KiCad/splitty/splitty.kicad_pcb (KiCad board)
At the start: 2 copper layers, 243.2 x 63.1 mm, 70 parts, among them U1 TRRS, U2 ProMicro, U3 ProMicro, U4 TRRS

Commit message: various fixes and changes
Parts:
- moved MX1 23.9 mm to (54.8, 123.3)
- moved MX32 23.9 mm to (238.3, 123.1)
- moved D1 23.9 mm to (54.7, 129.3)
- moved D32 23.9 mm to (238.3, 129.2)
- moved U4 11.8 mm to (48.8, 110.2), turned to 270 degrees
- moved U1 11.6 mm to (244.2, 109.9), turned to 90 degrees
- moved D4 7.37 mm to (66.8, 110.2)
- moved D31 7.37 mm to (226.2, 110.1)
Routing:
- net RCOL0: track 168.9 -> 185.3 mm
- net LGND: track 131.4 -> 141.1 mm
- net LDATA: track 153.9 -> 163.6 mm
- net RVCC: track 152.1 -> 157.9 mm
- net LVCC: track 137.1 -> 142.7 mm
- net RDATA: track 133.2 -> 138.6 mm
- net RGND: track 131.9 -> 136.2 mm
- net LROW0: track 243.0 -> 246.2 mm
- net Net-(D31-Pad2): track 11.2 -> 14.3 mm
- net Net-(D4-Pad2): track 11.2 -> 14.2 mm
- net Net-(D1-Pad2): track 13.9 -> 16.2 mm
- net RROW0: track 263.3 -> 262.1 mm
- added copper zone on B.Cu, net (none)
- removed copper zone on B.Cu, net LGND
Other:
- board size 243.2 x 63.1 mm -> 205 x 77.4 mm

Commit message: changed some shit i forget
Parts:
- removed D17, D18, D19, D20, D21, D22, D23, D24, D25, D26, D27, D28, D29, D30, D31, D32: D_Small, Keebio-Parts:Diode-dual
- removed G*** (x2): LOGO, Logos:tiny_lg_logo
- removed MX17, MX18, MX19, MX20, MX21, MX22, MX23, MX24, MX25, MX26, MX27, MX28, MX29, MX30, MX31, MX32: MX-NoLED, MX_Alps_Hybrid:MX-1U-NoLED
- removed U1, U4: TRRS, Keebio-Parts:TRRS-PJ-320A
- removed U3: ProMicro, promicro:ProMicro
- added J1: MJ-4PP-9-Lily58-cache, Footprints:TRRS_JACK_MJ4PP9, F.Cu at (244.3, 110.6)
- added JP1: Jumper, Footprints:ResetJumper, F.Cu at (157.5, 116.1)
- D1, D10, D11, D12, D13, D14, D15, D16, D2, D3, D4, D5, D6, D7, D8, D9: footprint Keebio-Parts:Diode-dual -> Footprints:Diode-dual; moved to F.Cu
- MX1, MX10, MX11, MX12, MX13, MX14, MX15, MX16, MX2, MX3, MX4, MX5, MX6, MX7, MX8, MX9: footprint MX_Alps_Hybrid:MX-1U-NoLED -> Footprints:reversible-mx-alps-choc
- U2: footprint promicro:ProMicro -> Footprints:ProMicro_v2; moved to F.Cu
- moved D1 192.2 mm to (246.9, 123.2), turned to 270 degrees
- moved MX1 183.5 mm to (238.3, 123.1)
- moved D11 106.7 mm to (223.1, 65.9), turned to 270 degrees
- moved D12 106.7 mm to (223.1, 85.1), turned to 270 degrees
- moved D14 106.7 mm to (242.2, 66.0), turned to 270 degrees
- moved D15 106.7 mm to (242.2, 85.1), turned to 270 degrees
- moved D2 106.7 mm to (166.0, 66.0), turned to 270 degrees
- moved D8 106.7 mm to (204.1, 66.0), turned to 270 degrees
- moved D5 106.7 mm to (185.0, 66.0), turned to 270 degrees
- moved D7 106.7 mm to (185.0, 104.1), turned to 270 degrees
- moved D6 106.6 mm to (185.0, 85.0), turned to 270 degrees
- moved D13 106.6 mm to (223.1, 104.1), turned to 270 degrees
- moved D10 106.6 mm to (204.1, 104.1), turned to 270 degrees
- moved D3 106.6 mm to (166.0, 85.1), turned to 270 degrees
- moved D9 106.6 mm to (204.1, 85.2), turned to 270 degrees
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Connections:
- net LCOL4 renamed COL3
- net LROW1 renamed ROW1
- D1 pad 1: LROW0 -> ROW2
- D10 pad 1: LROW0 -> ROW2
- D11 pad 1: LROW2 -> ROW0
- D13 pad 1: LROW0 -> ROW2
- D14 pad 1: LROW2 -> ROW0
- D16 pad 1: LROW0 -> ROW2
- D2 pad 1: LROW2 -> ROW0
- D4 pad 1: LROW0 -> ROW2
- D5 pad 1: LROW2 -> ROW0
- D7 pad 1: LROW0 -> ROW2
- D8 pad 1: LROW2 -> ROW0
- MX1 pad 1: LCOL0 -> COL5
- MX10 pad 1: LCOL3 -> COL2
- MX14 pad 1: LCOL5 -> COL4
- MX15 pad 1: LCOL5 -> COL4
- MX16 pad 1: LCOL5 -> COL4
- MX2 pad 1: LCOL1 -> COL0
- MX3 pad 1: LCOL1 -> COL0
- MX4 pad 1: LCOL1 -> COL0
- MX5 pad 1: LCOL2 -> COL1
- MX6 pad 1: LCOL2 -> COL1
- MX7 pad 1: LCOL2 -> COL1
- MX8 pad 1: LCOL3 -> COL2
- MX9 pad 1: LCOL3 -> COL2
- U2 pad 1: LDATA -> DATA
- U2 pad 11: Net-(U2-Pad11) -> COL4
- U2 pad 12: Net-(U2-Pad12) -> COL2
- U2 pad 14: LCOL3 -> COL5
- U2 pad 15: LCOL5 -> COL1
- U2 pad 16: LCOL2 -> Net-(U2-Pad16)
- U2 pad 17: LCOL1 -> Net-(U2-Pad17)
- U2 pad 18: LCOL0 -> ROW2
- U2 pad 20: LROW0 -> Net-(U2-Pad20)
- U2 pad 21: LVCC -> VCC
- U2 pad 23: LGND -> +5V
- U2 pad 3: LGND -> +5V
- U2 pad 4: Net-(U2-Pad4) -> +5V
- U2 pad 5: Net-(U2-Pad5) -> COL0
- U2 pad 6: LROW2 -> Net-(U2-Pad6)
- U2 pad 8: Net-(U2-Pad8) -> ROW0
Routing:
- net RROW0: track 262.1 -> 0.00 mm
- net LROW0: track 246.2 -> 0.00 mm
- net RROW1: track 223.6 -> 0.00 mm
- net RROW2: track 200.4 -> 0.00 mm
- net RCOL0: track 185.3 -> 0.00 mm
- net LDATA: track 163.6 -> 0.00 mm
- net LCOL0: track 159.5 -> 0.00 mm
- net RVCC: track 157.9 -> 0.00 mm
- net LVCC: track 142.7 -> 0.00 mm
- net COL4: track 0.00 -> 141.8 mm, vias 0 -> 1
- net LGND: track 141.1 -> 0.00 mm
- net RCOL1: track 140.6 -> 0.00 mm
- net RDATA: track 138.6 -> 0.00 mm
- net LCOL1: track 136.6 -> 0.00 mm
- net RGND: track 136.2 -> 0.00 mm
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- added copper zone on B.Cu, net +5V
- added copper zone on F.Cu, net +5V
- removed copper zone on B.Cu, net (none)
- removed copper zone on F.Cu, net LGND
- removed copper zone on B.Cu, net RGND
- removed copper zone on F.Cu, net RGND
Other:
- board size 205 x 77.4 mm -> 102.6 x 77.2 mm

Commit message: .
Routing:
- net DATA: track 116.5 -> 6.22 mm
- net +5V: track 115.5 -> 5.95 mm, vias 5 -> 0
- net VCC: track 109.8 -> 2.45 mm
- net COL4: track 141.8 -> 38.1 mm, vias 1 -> 0
- net COL5: track 94.8 -> 0.00 mm
- net COL3: track 116.6 -> 38.1 mm
- net COL2: track 97.5 -> 38.1 mm
- net COL0: track 106.2 -> 49.7 mm
- net ROW0: track 125.7 -> 81.4 mm
- net ROW2: track 120.7 -> 77.7 mm, vias 2 -> 0
- net Net-(JP1-Pad1): track 42.2 -> 0.00 mm
- net COL1: track 53.0 -> 19.1 mm
- net ROW1: track 105.1 -> 81.3 mm
- net Net-(D16-Pad2): track 14.5 -> 0.00 mm
- net Net-(D9-Pad2): track 9.03 -> 0.00 mm
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- removed copper zone on B.Cu, net +5V
- removed copper zone on F.Cu, net +5V

Commit message: .
.
Parts:
- removed J1: MJ-4PP-9-Lily58-cache, Footprints:TRRS_JACK_MJ4PP9
- added G***: LOGO, Footprints:size-matters-silk, F.Cu at (205.4, 114.0)
- added G***: LOGO, Footprints:size-matters-silk, B.Cu at (205.1, 114.0)
- added G***: LOGO, Footprints:3.7x3.7mm-lg-silk, F.Cu at (159.6, 116.2)
- added G***: LOGO, Footprints:3.7x3.7mm-lg-silk, B.Cu at (159.9, 116.2)
- added U1: ProMicro, Footprints:splitty-pro-micro, F.Cu at (165.0, 102.2)
- JP1: footprint Footprints:ResetJumper -> Footprints:splitty-reset-jumper
- U2: value ProMicro -> TRRS; footprint Footprints:ProMicro_v2 -> Footprints:TRRS_JACK_MJ4PP9
- moved D1 100.1 mm to (164.7, 66.0)
- moved MX1 99.2 mm to (157.2, 65.9)
- moved U2 80.4 mm to (244.3, 113.4), turned to 270 degrees
- moved D11 69.8 mm to (164.6, 103.8)
- moved MX11 68.7 mm to (157.2, 104.0)
- moved MX4 68.7 mm to (214.4, 65.9)
- moved D4 67.5 mm to (221.9, 66.0)
- moved MX5 57.1 mm to (233.4, 65.9)
- moved D5 55.9 mm to (240.9, 66.0)
- moved D12 43.8 mm to (183.8, 104.2)
- moved D14 43.1 mm to (221.9, 104.1)
- moved MX10 42.6 mm to (233.4, 85.0)
- moved MX12 42.6 mm to (176.3, 104.0)
- moved MX14 42.6 mm to (214.4, 104.0)
- moved MX3 42.6 mm to (195.3, 65.9)
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Connections:
- D1 pad 1: ROW2 -> ROW0
- D10 pad 1: ROW2 -> ROW1
- D11 pad 1: ROW0 -> ROW2
- D12 pad 1: ROW1 -> ROW2
- D14 pad 1: ROW0 -> ROW2
- D15 pad 1: ROW1 -> ROW2
- D3 pad 1: ROW1 -> ROW0
- D4 pad 1: ROW2 -> ROW0
- D7 pad 1: ROW2 -> ROW1
- D8 pad 1: ROW0 -> ROW1
- MX1 pad 1: COL5 -> COL0
- MX10 pad 1: COL2 -> COL4
- MX11 pad 1: COL3 -> COL0
- MX12 pad 1: COL3 -> COL1
- MX13 pad 1: COL3 -> COL2
- MX14 pad 1: COL4 -> COL3
- MX16 pad 1: COL4 -> COL5
- MX2 pad 1: COL0 -> COL1
- MX3 pad 1: COL0 -> COL2
- MX4 pad 1: COL0 -> COL3
- MX5 pad 1: COL1 -> COL4
- MX6 pad 1: COL1 -> COL0
- MX9 pad 1: COL2 -> COL3
- U2 pad 1: DATA -> SERIAL
- U2 pad 2: Net-(U2-Pad2) -> VCC
- U2 pad 4: +5V -> Net-(U2-Pad4)
Routing:
- net VCC: track 2.45 -> 125.1 mm
- net SERIAL: track 0.00 -> 105.9 mm
- net COL4: track 38.1 -> 124.0 mm
- net COL5: track 0.00 -> 83.6 mm, vias 0 -> 1
- net COL3: track 38.1 -> 110.8 mm
- net ROW1: track 81.3 -> 145.7 mm
- net Net-(JP1-Pad1): track 0.00 -> 49.5 mm
- net COL0: track 49.7 -> 97.8 mm
- net ROW0: track 81.4 -> 122.1 mm
- net ROW2: track 77.7 -> 117.2 mm
- net COL2: track 38.1 -> 71.3 mm
- net COL1: track 19.1 -> 48.9 mm
- net DATA: track 6.22 -> 0.00 mm
- net Net-(J1-Pad4): track 5.95 -> 0.00 mm
- net Net-(D12-Pad2): track 0.00 -> 5.83 mm
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- added copper zone on B.Cu, net +5V
- added copper zone on F.Cu, net +5V
Other:
- net class Power added: clearance 0.2, trace_width 0.381, via_dia 0.8, via_drill 0.4
