File: KiCad/splitty/splitty.sch (KiCad schematic (older format))
At the start: 68 parts, among them U1 TRRS, U2 ProMicro, U3 ProMicro, U4 TRRS

Commit message: changed some shit i forget
Parts:
- removed D1, D10, D11, D12, D13, D14, D15, D16, D17, D18, D19, D2, D20, D21, D22, D23, D24, D25, D26, D27, D28, D29, D3, D30, D31, D32, D4, D5, D6, D7, D8, D9: D_Small, Keebio-Parts:Diode-dual, symbol Device:D_Small
- removed MX1, MX10, MX11, MX12, MX13, MX14, MX15, MX16, MX17, MX18, MX19, MX2, MX20, MX21, MX22, MX23, MX24, MX25, MX26, MX27, MX28, MX29, MX3, MX30, MX31, MX32, MX4, MX5, MX6, MX7, MX8, MX9: MX-NoLED, MX_Alps_Hybrid:MX-1U-NoLED, symbol MX_Alps_Hybrid:MX-NoLED
- removed U1, U4: TRRS, Keebio-Parts:TRRS-PJ-320A, symbol keebio:TRRS
- removed U2, U3: ProMicro, promicro:ProMicro, symbol promicro:ProMicro

Commit message: .
.
Parts:
- added D1, D10, D11, D12, D13, D14, D15, D16, D2, D3, D4, D5, D6, D7, D8, D9: D_Small, Footprints:Diode-dual, symbol Device:D_Small
- added JP1: Jumper, Footprints:splitty-reset-jumper, symbol Device:Jumper
- added MX1, MX10, MX11, MX12, MX13, MX14, MX15, MX16, MX2, MX3, MX4, MX5, MX6, MX7, MX8, MX9: MX-NoLED, Footprints:reversible-mx-alps-choc, symbol MX_Alps_Hybrid:MX-NoLED
- added U1: ProMicro, Footprints:splitty-pro-micro, symbol promicro:ProMicro
- added U2: TRRS, Footprints:TRRS_JACK_MJ4PP9, symbol keebio:TRRS
Connections:
- new net: D1.2 (A), MX1.2 (ROW)
- new net: D2.2 (A), MX2.2 (ROW)
- new net: D3.2 (A), MX3.2 (ROW)
- new net: D4.2 (A), MX4.2 (ROW)
- new net: D5.2 (A), MX5.2 (ROW)
- new net: D6.2 (A), MX6.2 (ROW)
- new net: D7.2 (A), MX7.2 (ROW)
- new net: D8.2 (A), MX8.2 (ROW)
- new net: D9.2 (A), MX9.2 (ROW)
- new net: D10.2 (A), MX10.2 (ROW)
- new net: D11.2 (A), MX11.2 (ROW)
- new net: D12.2 (A), MX12.2 (ROW)
- new net: D13.2 (A), MX13.2 (ROW)
- new net: D14.2 (A), MX14.2 (ROW)
- new net: D15.2 (A), MX15.2 (ROW)
- new net: D16.2 (A), MX16.2 (ROW)
- new net: JP1.1, U1.22 (RST)
- new net +5V: JP1.2, U1.23 (GND), U1.3 (GND), U1.4 (GND), U2.3 (RING1)
- new net COL0: MX1.1 (COL), MX11.1 (COL), MX6.1 (COL), U1.20 (F4)
- new net COL1: MX12.1 (COL), MX2.1 (COL), MX7.1 (COL), U1.10 (E6)
- new net COL2: MX13.1 (COL), MX3.1 (COL), MX8.1 (COL), U1.13 (B6)
- new net COL3: MX14.1 (COL), MX4.1 (COL), MX9.1 (COL), U1.12 (B5)
- new net COL4: MX10.1 (COL), MX15.1 (COL), MX5.1 (COL), U1.9 (D7)
- new net COL5: MX16.1 (COL), U1.17 (F7)
- new net ROW0: D1.1 (K), D2.1 (K), D3.1 (K), D4.1 (K), D5.1 (K), U1.8 (C6)
- new net ROW1: D10.1 (K), D6.1 (K), D7.1 (K), D8.1 (K), D9.1 (K), U1.18 (F6)
- new net ROW2: D11.1 (K), D12.1 (K), D13.1 (K), D14.1 (K), D15.1 (K), D16.1 (K), U1.19 (F5)
- new net SERIAL: U1.1 (TX), U2.1 (SLEEVE)
- new net VCC: U1.21 (VCC), U2.2 (TIP)
- no-connect marks 0 -> 10
